Commit message: lidar and sonar added

File: src/sensors_demo/urdf/base.xacro (robot description, xacro)
@@ -2,8 +2,8 @@
 <robot name="base_demo" xmlns:xacro="http://www.ros.org/wiki/xacro">
     <xacro:property name="PI" value="3.14" />
-    <xacro:property name="vert_samples" value="1" />
-    <xacro:property name="hori_samples" value="5" />
-    <xacro:property name="vert_min_angle" value="-1" />
-    <xacro:property name="vert_max_angle" value="1" />
+    <xacro:property name="vert_samples" value="10" />
+    <xacro:property name="hori_samples" value="720" />
+    <xacro:property name="vert_min_angle" value="-5" />
+    <xacro:property name="vert_max_angle" value="5" />
     <xacro:property name="hori_min_angle" value="-30" />
     <xacro:property name="hori_max_angle" value="30" />
@@ -13,6 +13,12 @@
     <xacro:property name="lx" value="0.1" />
     <xacro:property name="ly" value="0.1" />
+<!---->
     <xacro:include filename="$(find sensors_demo)/urdf/materials.xacro" />
+    <xacro:include filename="$(find sensors_demo)/urdf/sonar.gazebo" />
+    <xacro:include filename="$(find sensors_demo)/urdf/lidar.gazebo" />
     <link name="root" />
+    <gazebo reference="base_link">
+       <material>Gazebo/RedBright</material>
+    </gazebo>
     <link name="base_link">
         <visual>
@@ -46,10 +52,8 @@
                 <cylinder radius="${lx/4}" length="${lx/2}"/>
             </geometry>
-            <material name="material_name">
-                <color rgba="1 1 1 1" />
-            </material>
+            <material name="pink"></material>
         </visual>
         <collision>
-            <origin xyz="0 0 ${lz/2}" rpy="0 0 0" />
+            <origin xyz="0 0 ${lz}" rpy="0 0 0" />
             <geometry>
                 <cylinder radius="${lx/4}" length="${lx/2}"/>
@@ -62,3 +66,9 @@
         </inertial>
     </link>
+    <joint name="sensor_joint" type="fixed">
+        <parent link="base_link" />
+        <child link="sensor_link" />
+        <origin xyz="0 0 ${lz}" rpy="0 0 0" />
+        <axis xyz="1 0 0" />
+    </joint>
 </robot>

File: src/sensors_demo/urdf/materials.xacro (robot description, xacro)
@@ -16,4 +16,7 @@
     <color rgba="${255/255} ${108/255} ${10/255} 1.0"/>
   </material>
+  <material name="pink">
+    <color rgba="${255/255} ${0/255} ${255/255} 1.0"/>
+  </material>
   <material name="brown">
     <color rgba="${222/255} ${207/255} ${195/255} 1.0"/>
