Commit message: sphere added

File: src/sensors_demo/urdf/geometric.xacro (robot description, xacro)
@@ -2,52 +2,78 @@
 <robot name="geom_demo" xmlns:xacro="http://www.ros.org/wiki/xacro">
     <xacro:property name="dens_alu" value="2712"/>
-    <xacro:property name="dens_au" value="19320"/>
+    <material name="green">
+        <color rgba="0 1 0 1"/>
+    </material>
+    <material name="blue">
+        <color rgba="0 0 1 1"/>
+    </material>
+    <material name="red">
+        <color rgba="1 0 0 1"/>
+    </material>
     <xacro:property name="cuboid_x" value="1.0"/>
     <xacro:property name="cuboid_y" value="1.0"/>
     <xacro:property name="cuboid_z" value="1.0"/>
     <xacro:property name="cuboid_m" value="${dens_alu * cuboid_x * cuboid_y * cuboid_z}" />
-    <xacro:property name="cuboid_Ix" value="${(1/12) * cuboid_m * (pow(cuboid_y, 2) + pow(cuboid_z, 2))}"/>
-    <xacro:property name="cuboid_Iy" value="${(1/12) * cuboid_m * (pow(cuboid_x, 2) + pow(cuboid_z, 2))}"/>
-    <xacro:property name="cuboid_Iz" value="${(1/12) * cuboid_m * (pow(cuboid_x, 2) + pow(cuboid_y, 2))}"/>
-    <material name="white">
-        <color rgba="0 1 0 1"/>
-    </material>
-<link name="cuboid">
-    <visual>
-        <origin xyz="0 0 ${cuboid_z/2}" rpy="0 0 0" />
-        <geometry>
-            <box size="${cuboid_x} ${cuboid_y} ${cuboid_z}" />
-        </geometry>
-        <material name="green" />
-    </visual>
-    <inertial>
-        <origin xyz="0 0 ${cuboid_z/2}" rpy="0 0 0" />
-        <mass value="${cuboid_m}" />
-        <inertia ixx="${cuboid_Ix}" ixy="0.0" ixz="0.0"
-                 iyy="${cuboid_Iy}" iyz="0.0"
-                 izz="${cuboid_Iz}" />
-    </inertial>
-</link>
-<xacro:property name="cylinder_r" value="1.0"/>
-<xacro:property name="cylinder_z" value="1.0"/>
-<xacro:property name="cylinder_m" value="${dens_alu * pi * pow(cylinder_r,2) * cylinder_z}"/>
-<xacro:property name="cylinder_Ix" value="${(1/12) * cylinder_m * (3 * pow(cylinder_r, 2) + pow(cylinder_z, 2))}"/>
-<xacro:property name="cylinder_Iy" value="${cylinder_Ix}"/>
-<xacro:property name="cylinder_Iz" value="${(1/2) * cylinder_m * pow(cylinder_r,2)}"/>
-<link name="cylinder">
-    <visual>
-        <origin xyz="0 0 ${cylinder_z/2}" rpy="0 0 0" />
-        <geometry>
-            <cylinder radius="${cylinder_r}" length="${cylinder_z}" />
-        </geometry>
-        <material name="green" />
-    </visual>
-    <inertial>
-        <origin xyz="0 0 ${cylinder_z/2}" rpy="0 0 0" />
-        <mass value="${cylinder_m}" />
-        <inertia ixx="${cylinder_Ix}" ixy="0.0" ixz="0.0"
-                 iyy="${cylinder_Iy}" iyz="0.0"
-                 izz="${cylinder_Iz}" />
-    </inertial>
-</link>
+    <xacro:property name="cuboid_Ix" value="${(1.0/12.0) * cuboid_m * (pow(cuboid_y, 2) + pow(cuboid_z, 2))}"/>
+    <xacro:property name="cuboid_Iy" value="${(1.0/12.0) * cuboid_m * (pow(cuboid_x, 2) + pow(cuboid_z, 2))}"/>
+    <xacro:property name="cuboid_Iz" value="${(1.0/12.0) * cuboid_m * (pow(cuboid_x, 2) + pow(cuboid_y, 2))}"/>
+    <link name="cuboid">
+        <visual>
+            <origin xyz="-2.5 0 ${cuboid_z/2}" rpy="0 0 0" />
+            <geometry>
+                <box size="${cuboid_x} ${cuboid_y} ${cuboid_z}" />
+            </geometry>
+            <material name="red" />
+        </visual>
+        <inertial>
+            <origin xyz="0 0 ${cuboid_z/2}" rpy="0 0 0" />
+            <mass value="${cuboid_m}" />
+            <inertia ixx="${cuboid_Ix}" ixy="0.0" ixz="0.0"
+                     iyy="${cuboid_Iy}" iyz="0.0"
+                     izz="${cuboid_Iz}" />
+        </inertial>
+    </link>
+    <xacro:property name="cylinder_r" value="1.0"/>
+    <xacro:property name="cylinder_z" value="1.0"/>
+    <xacro:property name="cylinder_m" value="${dens_alu * pi * pow(cylinder_r,2) * cylinder_z}"/>
+    <xacro:property name="cylinder_Ix" value="${(1.0/12.0) * cylinder_m * (3 * pow(cylinder_r, 2) + pow(cylinder_z, 2))}"/>
+    <xacro:property name="cylinder_Iy" value="${cylinder_Ix}"/>
+    <xacro:property name="cylinder_Iz" value="${(1.0/2.0) * cylinder_m * pow(cylinder_r,2)}"/>
+    <link name="cylinder">
+        <visual>
+            <origin xyz="0 0 ${cylinder_z/2}" rpy="0 0 0" />
+            <geometry>
+                <cylinder radius="${cylinder_r}" length="${cylinder_z}" />
+            </geometry>
+            <material name="green" />
+        </visual>
+        <inertial>
+            <origin xyz="0 0 ${cylinder_z/2}" rpy="0 0 0" />
+            <mass value="${cylinder_m}" />
+            <inertia ixx="${cylinder_Ix}" ixy="0.0" ixz="0.0"
+                     iyy="${cylinder_Iy}" iyz="0.0"
+                     izz="${cylinder_Iz}" />
+        </inertial>
+    </link>
+    <xacro:property name="sphere_r" value="1.0"/>
+    <xacro:property name="sphere_m" value="${dens_alu * (4.0/3.0) * pi * pow(sphere_r,3)}"/>
+    <xacro:property name="sphere_Ix" value="${(2.0/5.0) * sphere_m * pow(sphere_r, 2)}"/>
+    <xacro:property name="sphere_Iy" value="${(2.0/5.0) * sphere_m * pow(sphere_r, 2)}"/>
+    <xacro:property name="sphere_Iz" value="${(2.0/5.0) * sphere_m * pow(sphere_r, 2)}"/>
+    <link name="sphere">
+        <visual>
+            <origin xyz="2.5 0 ${sphere_r}" rpy="0 0 0" />
+            <geometry>
+                <sphere radius="${sphere_r}"/>
+            </geometry>
+            <material name="blue" />
+        </visual>
+        <inertial>
+            <origin xyz="0 0 ${sphere_r}" rpy="0 0 0" />
+            <mass value="${sphere_m}" />
+            <inertia ixx="${sphere_Ix}" ixy="0.0" ixz="0.0"
+                     iyy="${sphere_Iy}" iyz="0.0"
+                     izz="${sphere_Iz}" />
+        </inertial>
+    </link>
 </robot>
