Commit message: ros2 migrated

File: ros2_ws/src/sensors_demo/urdf/base.xacro (robot description, xacro)
@@ -1,23 +1,25 @@
 <?xml version="1.0"?>
 <robot name="base_demo" xmlns:xacro="http://www.ros.org/wiki/xacro">
+    <!-- Properties that can be used in the rest of the xacro file -->
     <xacro:property name="PI" value="3.14" />
     <xacro:property name="vert_samples" value="10" />
-    <xacro:property name="hori_samples" value="720" />
+    <xacro:property name="hori_samples" value="10" />
     <xacro:property name="vert_min_angle" value="-5" />
     <xacro:property name="vert_max_angle" value="5" />
+    <xacro:property name="hori_max_angle" value="30" />
     <xacro:property name="hori_min_angle" value="-30" />
-    <xacro:property name="hori_max_angle" value="30" />
-    <xacro:property name="range_min" value="0.1" />
+    <xacro:property name="range_min" value="1" />
     <xacro:property name="range_max" value="5.0" />
     <xacro:property name="lz" value="0.1" />
     <xacro:property name="lx" value="0.1" />
     <xacro:property name="ly" value="0.1" />
-<!---->
+    <!-- We can include other xacro or URDF files -->
     <xacro:include filename="$(find sensors_demo)/urdf/materials.xacro" />
-    <xacro:include filename="$(find sensors_demo)/urdf/sonar.gazebo" />
+    <!-- <xacro:include filename="$(find sensors_demo)/urdf/sonar.gazebo" /> -->
     <xacro:include filename="$(find sensors_demo)/urdf/lidar.gazebo" />
+    <!-- Rviz/Gazebo does not like the first link having mass or inertia, so a dummy link is created -->
     <link name="root" />
     <gazebo reference="base_link">
-       <material>Gazebo/RedBright</material>
+        <material>Gazebo/RedBright</material>
     </gazebo>
     <link name="base_link">
@@ -27,11 +29,10 @@
                 <box size="${lx} ${ly} ${lz}" />
             </geometry>
-            <material name="green">
-            </material>
+            <material name="green" />
         </visual>
         <collision>
             <origin xyz="0 0 ${lz/2}" rpy="0 0 0" />
             <geometry>
-                <box size="0.1 0.1 0.1" />
+                <box size="${lx} ${ly} ${lz}" />
             </geometry>
         </collision>
@@ -42,5 +43,5 @@
         </inertial>
     </link>
-    <joint name="root_link" type="fixed">
+    <joint name="root_joint" type="fixed">
         <parent link="root" />
         <child link="base_link" />
@@ -50,12 +51,12 @@
             <origin xyz="0 0 ${lz}" rpy="0 0 0" />
             <geometry>
-                <cylinder radius="${lx/4}" length="${lx/2}"/>
+                <cylinder radius="${lx/4}" length="${lz/2}" />
             </geometry>
-            <material name="pink"></material>
+            <material name="pink_i_guess" />
         </visual>
         <collision>
             <origin xyz="0 0 ${lz}" rpy="0 0 0" />
             <geometry>
-                <cylinder radius="${lx/4}" length="${lx/2}"/>
+                <cylinder radius="${lx/4}" length="${lz/2}" />
             </geometry>
         </collision>

File: ros2_ws/src/sensors_demo/urdf/materials.xacro (robot description, xacro)
@@ -16,6 +16,6 @@
     <color rgba="${255/255} ${108/255} ${10/255} 1.0"/>
   </material>
-  <material name="pink">
-    <color rgba="${255/255} ${0/255} ${255/255} 1.0"/>
+  <material name="pink_i_guess">
+    <color rgba="${255/255} ${0/255} ${128/255} 1.0"/>
   </material>
   <material name="brown">
